Commit message: checked customization colors on my own bot

File: TP3/robutler_description_tp3/urdf/common_properties.xacro (robot description, xacro)
@@ -29,4 +29,7 @@
     <color rgba="0.8 0.0 0.0 1.0"/>
   </material>
+  <material name="yellow">
+    <color rgba="0.8 0.8 0.0 1.0"/>
+  </material>
   <material name="white">
     <color rgba="1.0 1.0 1.0 1.0"/>

File: TP3/robutler_description_tp3/urdf/robutler.urdf.xacro (robot description, xacro)
@@ -15,5 +15,5 @@
         <mesh filename="package://turtlebot3_description/meshes/bases/waffle_pi_base.stl" scale="0.001 0.001 0.001"/>
       </geometry>
-      <material name="light_black"/>
+      <material name="red"/>
     </visual>
     <collision>
@@ -43,5 +43,5 @@
         <mesh filename="package://turtlebot3_description/meshes/wheels/left_tire.stl" scale="0.001 0.001 0.001"/>
       </geometry>
-      <material name="dark"/>
+      <material name="yellow"/>
     </visual>
     <collision>
@@ -71,5 +71,5 @@
         <mesh filename="package://turtlebot3_description/meshes/wheels/right_tire.stl" scale="0.001 0.001 0.001"/>
       </geometry>
-      <material name="dark"/>
+      <material name="yellow"/>
     </visual>
     <collision>
@@ -144,5 +144,5 @@
         <mesh filename="package://turtlebot3_description/meshes/sensors/lds.stl" scale="0.001 0.001 0.001"/>
       </geometry>
-      <material name="dark"/>
+      <material name="grey"/>
     </visual>
     <collision>
