Commit message: Ultimas alternações

File: robutler_description_tp3/urdf/common_properties.xacro (robot description, xacro)
@@ -15,5 +15,5 @@
   </material>
   <material name="green">
-    <color rgba="0.0 0.8 0.0 1.0"/>
+    <color rgba="0.7 0.2 0.2 1.0"/>
   </material>
   <material name="grey">
@@ -24,8 +24,11 @@
   </material>
   <material name="brown">
-    <color rgba="${222/255} ${207/255} ${195/255} 1.0"/>
+    <color rgba="0.7 0.2 0.2 1.0"/>
   </material>
   <material name="red">
     <color rgba="0.8 0.0 0.0 1.0"/>
+  </material>
+  <material name="yellow">
+    <color rgba="0.8 0.8 0.0 1.0"/>
   </material>
   <material name="white">

File: robutler_description_tp3/urdf/robutler.gazebo.xacro (robot description, xacro)
@@ -5,5 +5,5 @@
   <xacro:arg name="imu_visual"    default="false"/>
   <gazebo reference="base_link">
-    <material>Gazebo/LightBlue</material>
+    <material>Gazebo/Red</material>
   </gazebo>
   <gazebo reference="wheel_left_link">
@@ -15,5 +15,5 @@
     <maxVel>0.1</maxVel>
     <fdir1>1 0 0</fdir1>
-    <material>Gazebo/FlatBlack</material>
+    <material>Gazebo/ZincYellow</material>
   </gazebo>
   <gazebo reference="wheel_right_link">
@@ -25,5 +25,5 @@
     <maxVel>0.1</maxVel>
     <fdir1>1 0 0</fdir1>
-    <material>Gazebo/FlatBlack</material>
+    <material>Gazebo/Yellow</material>
   </gazebo>
   <gazebo reference="caster_back_right_link">
@@ -103,5 +103,5 @@
   </gazebo>
   <gazebo reference="base_scan">
-    <material>Gazebo/Blue</material>
+    <material>Gazebo/Grey</material>
     <sensor type="ray" name="lds_lfcd_sensor">
       <pose>0 0 0 0 0 0</pose>
@@ -168,4 +168,74 @@
     </sensor>
   </gazebo>
-                    <!-- COLOCAR CAMARA NA PARTE SUPERIOR -->
+                    <!-- COLOCAR CAMARA NA PARTE SUPERIOR / MINHAS ALTERAÇÕES-->
+  <gazebo reference="antena">
+    <material>Gazebo/WoodFloor</material>
+  </gazebo>
+  <gazebo reference="antena_link">
+    <material>Gazebo/Grey</material>
+  </gazebo>
+  <!-- <gazebo reference="top_scan">
+    <material>Gazebo/Red</material>
+    <sensor type="ray" name="lds_lfcd_sensor">
+      <pose>-0.150 0 2 0 0 0</pose>
+      <visualize>$(arg laser_visual)</visualize>
+      <update_rate>5</update_rate>
+      <ray>
+        <scan>
+          <horizontal>
+            <samples>360</samples>
+            <resolution>1</resolution>
+            <min_angle>0.0</min_angle>
+            <max_angle>6.28319</max_angle>
+          </horizontal>
+        </scan>
+        <range>
+          <min>0.100</min>
+          <max>1.5</max>
+          <resolution>0.015</resolution>
+        </range>
+        <noise>
+          <type>gaussian</type>
+          <mean>0.0</mean>
+          <stddev>0.01</stddev>
+        </noise>
+      </ray>
+      <plugin name="top_gazebo_ros_lds_lfcd_controller" filename="libgazebo_ros_laser.so">
+        <topicName>top_scan</topicName>
+        <frameName>top_scan</frameName>
+      </plugin>
+    </sensor>
+  </gazebo> -->
+  <gazebo reference="top_camera_rgb_frame">
+    <sensor type="camera" name="Pi Camera">
+      <always_on>true</always_on>
+      <visualize>$(arg camera_visual)</visualize>
+      <camera>
+          <horizontal_fov>1.085595</horizontal_fov>
+          <image>
+              <width>640</width>
+              <height>480</height>
+              <format>R8G8B8</format>
+          </image>
+          <clip>
+              <near>0.03</near>
+              <far>100</far>
+          </clip>
+      </camera>
+      <plugin name="top_camera_controller" filename="libgazebo_ros_camera.so">
+        <alwaysOn>true</alwaysOn>
+        <updateRate>30.0</updateRate>
+        <cameraName>camera</cameraName>
+        <frameName>top_camera_rgb_optical_frame</frameName>
+        <imageTopicName>rgb/top_image_raw</imageTopicName>
+        <cameraInfoTopicName>rgb/top_camera_info</cameraInfoTopicName>
+        <hackBaseline>0.07</hackBaseline>
+        <distortionK1>0.0</distortionK1>
+        <distortionK2>0.0</distortionK2>
+        <distortionK3>0.0</distortionK3>
+        <distortionT1>0.0</distortionT1>
+        <distortionT2>0.0</distortionT2>
+      </plugin>
+    </sensor>
+  </gazebo>
 </robot>

File: robutler_description_tp3/urdf/robutler.urdf.xacro (robot description, xacro)
@@ -185,3 +185,88 @@
   </joint>
   <link name="camera_rgb_optical_frame"/>
+<!-- Minhas alterações a partir daqui -->
+                                            <!-- Ver se esta antena pode ser rotativa pra camara -->
+  <link name="antena">
+    <visual>
+      <geometry>
+        <cylinder length="0.300" radius="0.01"/>
+      </geometry>
+      <origin xyz="0 0 0.122" rpy="0 0 0"/>
+      <!-- antes 0.122 -->
+      <material name="blue"/>
+    </visual>
+  </link>
+  <joint name="body_to_antena" type="fixed">
+    <parent link="base_link"/>
+    <child link="antena"/>
+    <origin xyz="-0.150 0 0.118" rpy="0 0 0"/>
+  </joint>
+  <link name="antena_link">
+    <visual>
+      <geometry>
+        <cylinder length="0.025" radius="0.05"/>
+      </geometry>
+      <origin xyz="0 0 0" rpy="0 0 0"/>
+      <material name="blue"/>
+    </visual>
+  </link>
+  <joint name="antena_to_antena_link" type="fixed">
+    <parent link="antena"/>
+    <child link="antena_link"/>
+    <origin xyz="0 0 0.275" rpy="0 0 0"/>
+  </joint>
+  <!-- SCAN -->
+  <!-- <link name="top_scan">
+    <visual>
+      <origin xyz="0 0 0" rpy="0 0 0"/>
+      <geometry>
+        <mesh filename="package://turtlebot3_description/meshes/sensors/lds.stl" scale="0.001 0.001 0.001"/>
+      </geometry>
+      <material name="dark"/>
+    </visual>
+    <collision>
+      <origin xyz="0.015 0 -0.0065" rpy="0 0 0"/>
+      <geometry>
+        <cylinder length="0.0315" radius="0.055"/>
+      </geometry>
+    </collision>
+    <inertial>
+      <mass value="0.114" />
+      <origin xyz="0 0 0" />
+      <inertia ixx="0.001" ixy="0.0" ixz="0.0"
+               iyy="0.001" iyz="0.0"
+               izz="0.001" />
+    </inertial>
+  </link>
+  <joint name="antena_link_to_top_scan" type="fixed">
+    <origin xyz="0 0 0" rpy="0 0 0"/>
+    <parent link="antena_link"/>
+    <child link="top_scan"/>
+  </joint> -->
+  <!-- CAMARA -->
+  <joint name="top_camera_joint" type="fixed">
+    <origin xyz="0.035 0 0" rpy="0 0 0"/>
+    <parent link="antena_link"/>
+    <child link="top_camera_link"/>
+  </joint>
+  <link name="top_camera_link">
+    <collision>
+      <origin xyz="0 0 0" rpy="0 0 0"/>
+      <geometry>
+        <box size="0.015 0.030 0.027"/>
+      </geometry>
+    </collision>
+  </link>
+  <joint name="top_camera_rgb_joint" type="fixed">
+    <origin xyz="0 0 0" rpy="0 0 0"/>
+    <parent link="top_camera_link"/>
+    <child link="top_camera_rgb_frame"/>
+  </joint>
+  <link name="top_camera_rgb_frame"/>
+  <joint name="top_camera_rgb_optical_joint" type="fixed">
+    <origin xyz="0 0 0" rpy="-1.57 0 -1.57"/>
+    <parent link="top_camera_rgb_frame"/>
+    <child link="top_camera_rgb_optical_frame"/>
+  </joint>
+  <link name="top_camera_rgb_optical_frame"/>
 </robot>
