Commit message: laptop detection is working properly, new camera added

File: robutler_description_tp3/urdf/robutler.gazebo.xacro (robot description, xacro)
@@ -239,3 +239,35 @@
     </sensor>
   </gazebo>
+  <gazebo reference="toptop_camera_rgb_frame">
+    <sensor type="camera" name="Pi Camera">
+      <always_on>true</always_on>
+      <visualize>$(arg camera_visual)</visualize>
+      <camera>
+          <horizontal_fov>1.085595</horizontal_fov>
+          <image>
+              <width>1920</width>
+              <height>1080</height>
+              <format>R8G8B8</format>
+          </image>
+          <clip>
+              <near>0.03</near>
+              <far>100</far>
+          </clip>
+      </camera>
+      <plugin name="toptop_camera_controller" filename="libgazebo_ros_camera.so">
+        <alwaysOn>true</alwaysOn>
+        <updateRate>30.0</updateRate>
+        <cameraName>camera</cameraName>
+        <frameName>toptop_camera_rgb_optical_frame</frameName>
+        <imageTopicName>rgb/toptop_image_raw</imageTopicName>
+        <cameraInfoTopicName>rgb/toptop_camera_info</cameraInfoTopicName>
+        <hackBaseline>0.07</hackBaseline>
+        <distortionK1>0.0</distortionK1>
+        <distortionK2>0.0</distortionK2>
+        <distortionK3>0.0</distortionK3>
+        <distortionT1>0.0</distortionT1>
+        <distortionT2>0.0</distortionT2>
+      </plugin>
+    </sensor>
+  </gazebo>
 </robot>

File: robutler_description_tp3/urdf/robutler.urdf.xacro (robot description, xacro)
@@ -270,3 +270,29 @@
   </joint>
   <link name="top_camera_rgb_optical_frame"/>
+  <!-- CAMARA -->
+  <joint name="toptop_camera_joint" type="fixed">
+    <origin xyz="0.035 0 0.6" rpy="0 0 0"/>
+    <parent link="antena_link"/>
+    <child link="toptop_camera_link"/>
+  </joint>
+  <link name="toptop_camera_link">
+    <collision>
+      <origin xyz="0 0 0" rpy="0 0 0"/>
+      <geometry>
+        <box size="0.015 0.030 0.027"/>
+      </geometry>
+    </collision>
+  </link>
+  <joint name="toptop_camera_rgb_joint" type="fixed">
+    <origin xyz="0 0 0" rpy="0 0 0"/>
+    <parent link="toptop_camera_link"/>
+    <child link="toptop_camera_rgb_frame"/>
+  </joint>
+  <link name="toptop_camera_rgb_frame"/>
+  <joint name="toptop_camera_rgb_optical_joint" type="fixed">
+    <origin xyz="0 0 0" rpy="-1.57 0 -1.57"/>
+    <parent link="toptop_camera_rgb_frame"/>
+    <child link="toptop_camera_rgb_optical_frame"/>
+  </joint>
+  <link name="toptop_camera_rgb_optical_frame"/>
 </robot>

Commit message: Search for coke/objects progress

File: robutler_description_tp3/urdf/robutler.gazebo.xacro (robot description, xacro)
@@ -239,3 +239,35 @@
     </sensor>
   </gazebo>
+  <gazebo reference="toptop_camera_rgb_frame">
+    <sensor type="camera" name="Pi Camera">
+      <always_on>true</always_on>
+      <visualize>$(arg camera_visual)</visualize>
+      <camera>
+          <horizontal_fov>1.085595</horizontal_fov>
+          <image>
+              <width>1920</width>
+              <height>1080</height>
+              <format>R8G8B8</format>
+          </image>
+          <clip>
+              <near>0.03</near>
+              <far>100</far>
+          </clip>
+      </camera>
+      <plugin name="toptop_camera_controller" filename="libgazebo_ros_camera.so">
+        <alwaysOn>true</alwaysOn>
+        <updateRate>30.0</updateRate>
+        <cameraName>camera</cameraName>
+        <frameName>toptop_camera_rgb_optical_frame</frameName>
+        <imageTopicName>rgb/toptop_image_raw</imageTopicName>
+        <cameraInfoTopicName>rgb/toptop_camera_info</cameraInfoTopicName>
+        <hackBaseline>0.07</hackBaseline>
+        <distortionK1>0.0</distortionK1>
+        <distortionK2>0.0</distortionK2>
+        <distortionK3>0.0</distortionK3>
+        <distortionT1>0.0</distortionT1>
+        <distortionT2>0.0</distortionT2>
+      </plugin>
+    </sensor>
+  </gazebo>
 </robot>

File: robutler_description_tp3/urdf/robutler.urdf.xacro (robot description, xacro)
@@ -244,5 +244,5 @@
     <child link="top_scan"/>
   </joint> -->
-  <!-- CAMARA -->
+  <!-- TOP CAMARA -->
   <joint name="top_camera_joint" type="fixed">
     <origin xyz="0.035 0 0" rpy="0 0 0"/>
@@ -270,3 +270,29 @@
   </joint>
   <link name="top_camera_rgb_optical_frame"/>
+    <!-- TOPTOPCAMARA -->
+  <joint name="toptop_camera_joint" type="fixed">
+    <origin xyz="0.035 0 0.6" rpy="0 0 0"/>
+    <parent link="antena_link"/>
+    <child link="toptop_camera_link"/>
+  </joint>
+  <link name="toptop_camera_link">
+    <collision>
+      <origin xyz="0 0 0" rpy="0 0 0"/>
+      <geometry>
+        <box size="0.015 0.030 0.027"/>
+      </geometry>
+    </collision>
+  </link>
+  <joint name="toptop_camera_rgb_joint" type="fixed">
+    <origin xyz="0 0 0" rpy="0 0 0"/>
+    <parent link="toptop_camera_link"/>
+    <child link="toptop_camera_rgb_frame"/>
+  </joint>
+  <link name="toptop_camera_rgb_frame"/>
+  <joint name="toptop_camera_rgb_optical_joint" type="fixed">
+    <origin xyz="0 0 0" rpy="-1.57 0 -1.57"/>
+    <parent link="toptop_camera_rgb_frame"/>
+    <child link="toptop_camera_rgb_optical_frame"/>
+  </joint>
+  <link name="toptop_camera_rgb_optical_frame"/>
 </robot>
