Commit message: Alteração de cor no rviz igual ao gazebo

File: robutler_description_tp3/urdf/robutler.urdf.xacro (robot description, xacro)
@@ -15,5 +15,5 @@
         <mesh filename="package://turtlebot3_description/meshes/bases/waffle_pi_base.stl" scale="0.001 0.001 0.001"/>
       </geometry>
-      <material name="light_black"/>
+      <material name="red"/>
     </visual>
     <collision>
@@ -43,5 +43,5 @@
         <mesh filename="package://turtlebot3_description/meshes/wheels/left_tire.stl" scale="0.001 0.001 0.001"/>
       </geometry>
-      <material name="dark"/>
+      <material name="yellow"/>
     </visual>
     <collision>
@@ -71,5 +71,5 @@
         <mesh filename="package://turtlebot3_description/meshes/wheels/right_tire.stl" scale="0.001 0.001 0.001"/>
       </geometry>
-      <material name="dark"/>
+      <material name="yellow"/>
     </visual>
     <collision>
@@ -144,5 +144,5 @@
         <mesh filename="package://turtlebot3_description/meshes/sensors/lds.stl" scale="0.001 0.001 0.001"/>
       </geometry>
-      <material name="dark"/>
+      <material name="grey"/>
     </visual>
     <collision>
@@ -194,5 +194,5 @@
       <origin xyz="0 0 0.122" rpy="0 0 0"/>
       <!-- antes 0.122 -->
-      <material name="blue"/>
+      <material name="brown"/>
     </visual>
   </link>
@@ -208,5 +208,5 @@
       </geometry>
       <origin xyz="0 0 0" rpy="0 0 0"/>
-      <material name="blue"/>
+      <material name="grey"/>
     </visual>
   </link>

Commit message: rviz color correction !

File: robutler_description_tp3/urdf/robutler.urdf.xacro (robot description, xacro)
@@ -15,5 +15,5 @@
         <mesh filename="package://turtlebot3_description/meshes/bases/waffle_pi_base.stl" scale="0.001 0.001 0.001"/>
       </geometry>
-      <material name="light_black"/>
+      <material name="red"/>
     </visual>
     <collision>
@@ -43,5 +43,5 @@
         <mesh filename="package://turtlebot3_description/meshes/wheels/left_tire.stl" scale="0.001 0.001 0.001"/>
       </geometry>
-      <material name="dark"/>
+      <material name="yellow"/>
     </visual>
     <collision>
@@ -71,5 +71,5 @@
         <mesh filename="package://turtlebot3_description/meshes/wheels/right_tire.stl" scale="0.001 0.001 0.001"/>
       </geometry>
-      <material name="dark"/>
+      <material name="yellow"/>
     </visual>
     <collision>
@@ -144,5 +144,5 @@
         <mesh filename="package://turtlebot3_description/meshes/sensors/lds.stl" scale="0.001 0.001 0.001"/>
       </geometry>
-      <material name="dark"/>
+      <material name="grey"/>
     </visual>
     <collision>
@@ -193,5 +193,5 @@
       <origin xyz="0 0 0.122" rpy="0 0 0"/>
       <!-- antes 0.122 -->
-      <material name="blue"/>
+      <material name="brown"/>
     </visual>
   </link>
@@ -207,5 +207,5 @@
       </geometry>
       <origin xyz="0 0 0" rpy="0 0 0"/>
-      <material name="blue"/>
+      <material name="grey"/>
     </visual>
   </link>
